Commit message: add joint limits and readme

File: config/L_JEARM.urdf (robot description, URDF)
Before this commit: robot L_JEARM, 8 links, 7 joints
Joints:
- joint joint1: limit lower=-5.14 upper=5.14 effort=100 velocity=3.14 -> lower=-3.14 upper=3.14 effort=100 velocity=3.14
- joint joint2: limit lower=-2.96 upper=2.96 effort=100 velocity=3.14 -> lower=-1.85 upper=1.8 effort=100 velocity=3.14
- joint joint4: limit lower=-2.27 upper=1.8 effort=100 velocity=3.14 -> lower=-2.26 upper=1.82 effort=100 velocity=3.14
