Commit message: change urdf and add diagnose

File: config/DUAL_JEARM.urdf (robot description, URDF)
Before this commit: robot DOUB_JEARM, 15 links, 14 joints
Links:
- added link left_base
- added link right_base
Joints:
- added joint left_base_joint: type fixed, parent base_link, child left_base, origin xyz=-0.0445 -0.2126 0.9008 rpy=1.5708 -1.5708 0
- added joint right_base_joint: type fixed, parent base_link, child right_base, origin xyz=-0.0445 0.2126 0.9008 rpy=1.5708 -1.5708 0
- joint joint11: origin xyz=-0.0445 -0.2126 0.9008 rpy=1.5708 -1.5708 0 -> xyz=0 0 0 rpy=0 0 0; parent base_link -> left_base
- joint joint12: origin xyz=0 0 0 rpy=-1.5708 0 0 -> xyz=-0.003618304232 0.002800664499 -0.000020332110 rpy=-1.578055952076 0.001477645909 -0.000010727340
- joint joint13: origin xyz=0 -0.2719 0 rpy=1.5708 0 0 -> xyz=0.002577761227 -0.271180901646 0.002201772484 rpy=1.562677256935 0.003380507847 -0.000027447130
- joint joint14: origin xyz=-0.008 0 0 rpy=-1.5708 0 0 -> xyz=-0.008039033242 0.000263254982 -0.000000669832 rpy=-1.573340747986 0.001973845457 -0.000005022302
- joint joint15: origin xyz=0.008 -0.2189 0 rpy=1.5708 0 0 -> xyz=0.007549404638 -0.219291199652 -0.000810881595 rpy=1.574494058691 -0.002310478327 -0.000008543561
- joint joint16: origin xyz=0 0 0 rpy=-1.5708 0 0 -> xyz=0.000169969851 0.001161741697 -0.000003374674 rpy=-1.573702441570 0.029711882558 -0.000086333680
- joint joint17: origin xyz=0 -0.124 0 rpy=1.5708 0 0 -> xyz=-0.000213373503 -0.129044569401 -0.000248313607 rpy=1.572720684130 -0.010830083632 -0.000020840569
- joint joint21: origin xyz=-0.0445 0.2126 0.9008 rpy=1.5708 -1.5708 0 -> xyz=0 0 0 rpy=0 0 0; parent base_link -> right_base
- joint joint22: origin xyz=0 0 0 rpy=1.5708 0 0 -> xyz=-0.002432052083 0.002185646404 0.000015291728 rpy=1.577793055631 -0.010832281600 -0.000075790291
- joint joint23: origin xyz=0 -0.2719 0 rpy=-1.5708 0 0 -> xyz=0.001734034519 -0.270155238592 0.006269796108 rpy=-1.594000958131 -0.007617614448 0.000176793957
- joint joint24: origin xyz=-0.008 0 0 rpy=1.5708 0 0 -> xyz=-0.008052611788 -0.000617648529 -0.000001194446 rpy=1.572730887114 0.026955963719 0.000052141688
- joint joint25: origin xyz=0.008 -0.2189 0 rpy=-1.5708 0 0 -> xyz=0.008322677408 -0.218695828883 -0.000046340328 rpy=-1.570584385430 0.021148517040 0.000004481912
- joint joint26: origin xyz=0 0 0 rpy=1.5708 0 0 -> xyz=0.000260228939 -0.000186710496 -0.000000041703 rpy=1.571019733087 -0.020689877062 -0.000004621919
- joint joint27: origin xyz=0 -0.124 0 rpy=-1.5708 0 0 -> xyz=-0.000623537028 -0.129477191461 0.000055933872 rpy=-1.571232110251 -0.131905287446 0.000057315602

Commit message: change urdf

File: config/DUAL_JEARM.urdf (robot description, URDF)
Before this commit: robot DOUB_JEARM, 17 links, 16 joints
Joints:
- joint joint12: origin xyz=-0.003618304232 0.002800664499 -0.000020332110 rpy=-1.578055952076 0.001477645909 -0.000010727340 -> xyz=-0.000373149555 0.001900253350 -0.000010536402 rpy=-1.576341075806 0.005047906924 -0.000027989545
- joint joint13: origin xyz=0.002577761227 -0.271180901646 0.002201772484 rpy=1.562677256935 0.003380507847 -0.000027447130 -> xyz=0.000067207243 -0.274477151543 0.001249511048 rpy=1.566243931566 0.006458272070 -0.000029400606
- joint joint14: origin xyz=-0.008039033242 0.000263254982 -0.000000669832 rpy=-1.573340747986 0.001973845457 -0.000005022302 -> xyz=-0.008712672083 0.001412086038 -0.000002369272 rpy=-1.572474178934 -0.001244432352 0.000002087975
- joint joint15: origin xyz=0.007549404638 -0.219291199652 -0.000810881595 rpy=1.574494058691 -0.002310478327 -0.000008543561 -> xyz=0.008588707987 -0.218745273184 -0.000144383338 rpy=1.571456379349 0.000908280101 0.000000599513
- joint joint16: origin xyz=0.000169969851 0.001161741697 -0.000003374674 rpy=-1.573702441570 0.029711882558 -0.000086333680 -> xyz=0.000256032326 0.000377161557 -0.000000662225 rpy=-1.572553168752 0.034269927934 -0.000060195125
- joint joint17: origin xyz=-0.000213373503 -0.129044569401 -0.000248313607 rpy=1.572720684130 -0.010830083632 -0.000020840569 -> xyz=-0.000460121091 -0.129585515026 -0.000149116049 rpy=1.571947153914 -0.013964895086 -0.000016070665
- joint joint22: origin xyz=-0.002432052083 0.002185646404 0.000015291728 rpy=1.577793055631 -0.010832281600 -0.000075790291 -> xyz=-0.001222442969 0.000952364065 0.000007536879 rpy=1.578710523928 -0.011225289527 -0.000088839143
- joint joint23: origin xyz=0.001734034519 -0.270155238592 0.006269796108 rpy=-1.594000958131 -0.007617614448 0.000176793957 -> xyz=0.001465436550 -0.271467816884 0.005610099415 rpy=-1.591459779466 -0.007585632176 0.000156766159
- joint joint24: origin xyz=-0.008052611788 -0.000617648529 -0.000001194446 rpy=1.572730887114 0.026955963719 0.000052141688 -> xyz=-0.008164975845 0.000859548671 0.000002615866 rpy=1.573840782444 0.027643232297 0.000084148137
- joint joint25: origin xyz=0.008322677408 -0.218695828883 -0.000046340328 rpy=-1.570584385430 0.021148517040 0.000004481912 -> xyz=0.008402057960 -0.218933139956 0.000814810680 rpy=-1.574518845465 0.020769951530 -0.000077311330
- joint joint26: origin xyz=0.000260228939 -0.000186710496 -0.000000041703 rpy=1.571019733087 -0.020689877062 -0.000004621919 -> xyz=-0.000308251772 -0.000261606426 -0.000000444734 rpy=1.572496762070 -0.022320868749 -0.000037952078
- joint joint27: origin xyz=-0.000623537028 -0.129477191461 0.000055933872 rpy=-1.571232110251 -0.131905287446 0.000057315602 -> xyz=-0.000221173522 -0.129403801882 0.000067238833 rpy=-1.571320486187 -0.131924874924 0.000068949261

Commit message: add logs

File: config/DUAL_JEARM.urdf (robot description, URDF)
Before this commit: robot DOUB_JEARM, 17 links, 16 joints
Joints:
- joint joint11: limit lower=-3.14 upper=3.14 effort=100 velocity=3.14 -> lower=-5.1400 upper=5.1400 effort=100 velocity=3.9800; origin xyz=0 0 0 rpy=0 0 0 -> xyz=0.000000 0.000000 0.000000 rpy=0.000000 -0.000000 0.000000
- joint joint12: limit lower=-1.85 upper=1.8 effort=100 velocity=3.14 -> lower=-1.7535 upper=1.7700 effort=100 velocity=3.9800; origin xyz=-0.000373149555 0.001900253350 -0.000010536402 rpy=-1.576341075806 0.005047906924 -0.000027989545 -> xyz=-0.000300 0.001900 -0.000009 rpy=-1.576396 0.005000 -0.000028
- joint joint13: limit lower=-2.96 upper=2.96 effort=100 velocity=3.14 -> lower=-2.9600 upper=2.9600 effort=100 velocity=5.5500; origin xyz=0.000067207243 -0.274477151543 0.001249511048 rpy=1.566243931566 0.006458272070 -0.000029400606 -> xyz=0.000067 -0.274597 0.001235 rpy=1.566296 0.006400 -0.000029
- joint joint14: limit lower=-2.26 upper=1.82 effort=100 velocity=3.14 -> lower=-2.2284 upper=1.7679 effort=100 velocity=5.5500; origin xyz=-0.008712672083 0.001412086038 -0.000002369272 rpy=-1.572474178934 -0.001244432352 0.000002087975 -> xyz=-0.000009 0.001400 -0.000003 rpy=-1.572596 -0.001200 0.000002
- joint joint15: limit lower=-2.96 upper=2.96 effort=100 velocity=3.14 -> lower=-2.9600 upper=2.9600 effort=100 velocity=5.5500; origin xyz=0.008588707987 -0.218745273184 -0.000144383338 rpy=1.571456379349 0.000908280101 0.000000599513 -> xyz=0.000009 -0.218700 -0.000153 rpy=1.571496 0.000900 0.000001
- joint joint16: limit lower=-1.6 upper=1.55 effort=100 velocity=3.14 -> lower=-1.5631 upper=1.4637 effort=100 velocity=5.5500; origin xyz=0.000256032326 0.000377161557 -0.000000662225 rpy=-1.572553168752 0.034269927934 -0.000060195125 -> xyz=0.000200 0.000400 -0.000008 rpy=-1.572597 0.034300 -0.000062
- joint joint17: limit lower=-2.96 upper=2.96 effort=100 velocity=3.14 -> lower=-2.9600 upper=2.9600 effort=100 velocity=5.8600; origin xyz=-0.000460121091 -0.129585515026 -0.000149116049 rpy=1.571947153914 -0.013964895086 -0.000016070665 -> xyz=-0.000500 -0.129600 -0.000163 rpy=1.571996 -0.014000 -0.000017
- joint joint21: limit lower=-5.14 upper=5.14 effort=100 velocity=3.14 -> lower=-5.1400 upper=5.1400 effort=100 velocity=3.9800; origin xyz=0 0 0 rpy=0 0 0 -> xyz=0.000000 0.000000 0.000000 rpy=0.000000 -0.000000 0.000000
- joint joint22: limit lower=-1.86 upper=1.82 effort=100 velocity=3.14 -> lower=-1.8100 upper=1.8100 effort=100 velocity=3.9800; origin xyz=-0.001222442969 0.000952364065 0.000007536879 rpy=1.578710523928 -0.011225289527 -0.000088839143 -> xyz=-0.001200 0.000900 -0.000006 rpy=1.578797 -0.011200 -0.000090
- joint joint23: limit lower=-2.96 upper=2.96 effort=100 velocity=3.14 -> lower=-3.1400 upper=3.1400 effort=100 velocity=5.5500; origin xyz=0.001465436550 -0.271467816884 0.005610099415 rpy=-1.591459779466 -0.007585632176 0.000156766159 -> xyz=0.001400 -0.271542 0.005632 rpy=-1.591497 -0.007498 0.000155
- joint joint24: limit lower=-2.27 upper=1.8 effort=100 velocity=3.14 -> lower=-2.2000 upper=1.8000 effort=100 velocity=5.5500; origin xyz=-0.008164975845 0.000859548671 0.000002615866 rpy=1.573840782444 0.027643232297 0.000084148137 -> xyz=-0.000008 0.000800 0.000003 rpy=1.573898 0.027600 0.000086
- joint joint25: limit lower=-2.96 upper=2.96 effort=100 velocity=3.14 -> lower=-3.1400 upper=3.1400 effort=100 velocity=5.5500; origin xyz=0.008402057960 -0.218933139956 0.000814810680 rpy=-1.574518845465 0.020769951530 -0.000077311330 -> xyz=0.000008 -0.218898 0.000832 rpy=-1.574597 0.020700 -0.000079
- joint joint26: limit lower=-1.6 upper=1.55 effort=100 velocity=3.14 -> lower=-1.5800 upper=1.5400 effort=100 velocity=5.5500; origin xyz=-0.000308251772 -0.000261606426 -0.000000444734 rpy=1.572496762070 -0.022320868749 -0.000037952078 -> xyz=-0.000300 -0.000200 -0.000007 rpy=1.572497 -0.022300 -0.000038
- joint joint27: limit lower=-2.96 upper=2.96 effort=100 velocity=3.14 -> lower=-3.1400 upper=3.1400 effort=100 velocity=5.8600; origin xyz=-0.000221173522 -0.129403801882 0.000067238833 rpy=-1.571320486187 -0.131924874924 0.000068949261 -> xyz=-0.000198 -0.129400 0.000051 rpy=-1.571402 -0.131900 0.000080

Commit message: new mdh para

File: config/DUAL_JEARM.urdf (robot description, URDF)
Before this commit: robot DOUB_JEARM, 17 links, 16 joints
Joints:
- joint joint12: origin xyz=-0.000300 0.001900 -0.000009 rpy=-1.576396 0.005000 -0.000028 -> xyz=-0.000022 0.000819 -0.000010 rpy=-1.582783 0.008827 -0.000106
- joint joint13: origin xyz=0.000067 -0.274597 0.001235 rpy=1.566296 0.006400 -0.000029 -> xyz=0.000105 -0.271736 -0.001654 rpy=1.576885 0.024570 0.000150
- joint joint14: origin xyz=-0.000009 0.001400 -0.000003 rpy=-1.572596 -0.001200 0.000002 -> xyz=-0.007792 0.000809 0.000002 rpy=-1.568882 0.001903 0.000004
- joint joint15: origin xyz=0.000009 -0.218700 -0.000153 rpy=1.571496 0.000900 0.000001 -> xyz=0.008004 -0.219279 -0.000748 rpy=1.574210 0.019075 0.000065
- joint joint16: origin xyz=0.000200 0.000400 -0.000008 rpy=-1.572597 0.034300 -0.000062 -> xyz=-0.000127 0.000033 0.000000 rpy=-1.570240 0.023953 0.000013
- joint joint17: origin xyz=-0.000500 -0.129600 -0.000163 rpy=1.571996 -0.014000 -0.000017 -> xyz=-0.000340 -0.128509 0.000605 rpy=1.566088 -0.026226 0.000123

File: config/L_JEARM.urdf (robot description, URDF)
Before this commit: robot L_JEARM, 8 links, 7 joints
Joints:
- joint joint2: origin xyz=0 0 0 rpy=-1.5708 0 0 -> xyz=-0.000022 0.000819 -0.000010 rpy=-1.582783 0.008827 -0.000106
- joint joint3: origin xyz=0 -0.2719 0 rpy=1.5708 0 0 -> xyz=0.000105 -0.271736 -0.001654 rpy=1.576885 0.024570 0.000150
- joint joint4: origin xyz=-0.008 0 0 rpy=-1.5708 0 0 -> xyz=-0.007792 0.000809 0.000002 rpy=-1.568882 0.001903 0.000004
- joint joint5: origin xyz=0.008 -0.2189 0 rpy=1.5708 0 0 -> xyz=0.008004 -0.219279 -0.000748 rpy=1.574210 0.019075 0.000065
- joint joint6: origin xyz=0 0 0 rpy=-1.5708 0 0 -> xyz=-0.000127 0.000033 0.000000 rpy=-1.570240 0.023953 0.000013
- joint joint7: origin xyz=0 -0.124 0 rpy=1.5708 0 0 -> xyz=-0.000340 -0.128509 0.000605 rpy=1.566088 -0.026226 0.000123

Commit message: change urdf to suit modify

File: config/DUAL_JEARM.urdf (robot description, URDF)
Before this commit: robot DOUB_JEARM, 17 links, 16 joints
Joints:
- joint joint12: origin xyz=-0.000022 0.000819 -0.000010 rpy=-1.582783 0.008827 -0.000106 -> xyz=-0.000022 0.000800 -0.000010 rpy=-1.582897 0.008799 -0.000106
- joint joint13: origin xyz=0.000105 -0.271736 -0.001654 rpy=1.576885 0.024570 0.000150 -> xyz=0.000100 -0.271795 -0.001685 rpy=1.576998 0.024600 0.000153
- joint joint14: origin xyz=-0.007792 0.000809 0.000002 rpy=-1.568882 0.001903 0.000004 -> xyz=-0.007800 0.000800 0.000001 rpy=-1.568996 0.001900 0.000003
- joint joint15: origin xyz=0.008004 -0.219279 -0.000748 rpy=1.574210 0.019075 0.000065 -> xyz=0.008000 -0.219299 -0.000768 rpy=1.574297 0.019100 0.000067
- joint joint16: origin xyz=-0.000127 0.000033 0.000000 rpy=-1.570240 0.023953 0.000013 -> xyz=-0.000100 0.000033 0.000000 rpy=-1.570296 0.023900 0.000012
- joint joint17: origin xyz=-0.000340 -0.128509 0.000605 rpy=1.566088 -0.026226 0.000123 -> xyz=-0.000300 -0.128499 0.000604 rpy=1.566095 -0.026200 0.000123
- joint joint22: origin xyz=-0.001200 0.000900 -0.000006 rpy=1.578797 -0.011200 -0.000090 -> xyz=-0.001200 0.000900 0.000007 rpy=1.578797 -0.011200 -0.000090
- joint joint23: origin xyz=0.001400 -0.271542 0.005632 rpy=-1.591497 -0.007498 0.000155 -> xyz=0.001400 -0.271542 0.005622 rpy=-1.591497 -0.007498 0.000155
- joint joint24: origin xyz=-0.000008 0.000800 0.000003 rpy=1.573898 0.027600 0.000086 -> xyz=-0.000008 0.000800 0.000002 rpy=1.573898 0.027600 0.000086
- joint joint26: origin xyz=-0.000300 -0.000200 -0.000007 rpy=1.572497 -0.022300 -0.000038 -> xyz=-0.000300 -0.000200 -0.000000 rpy=1.572497 -0.022300 -0.000038
- joint joint27: origin xyz=-0.000198 -0.129400 0.000051 rpy=-1.571402 -0.131900 0.000080 -> xyz=-0.000200 -0.129400 0.000078 rpy=-1.571402 -0.131900 0.000080
