Commit message: dual arm settings

File: config/right/R_JEARM.urdf (robot description, URDF)
Before this commit: robot L_JEARM, 8 links, 7 joints
Links:
- link Link1: geometry collision mesh filename=package://my_jearm_moveit_config/config/meshes/right/r_link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; visual mesh filename=package://my_jearm_moveit_config/config/meshes/right/r_link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
- link Link2: geometry collision mesh filename=package://my_jearm_moveit_config/config/meshes/right/r_link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; visual mesh filename=package://my_jearm_moveit_config/config/meshes/right/r_link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
- link Link3: geometry collision mesh filename=package://my_jearm_moveit_config/config/meshes/right/r_link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; visual mesh filename=package://my_jearm_moveit_config/config/meshes/right/r_link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
- link Link4: geometry collision mesh filename=package://my_jearm_moveit_config/config/meshes/right/r_link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; visual mesh filename=package://my_jearm_moveit_config/config/meshes/right/r_link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
- link Link5: geometry collision mesh filename=package://my_jearm_moveit_config/config/meshes/right/r_link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; visual mesh filename=package://my_jearm_moveit_config/config/meshes/right/r_link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
- link Link6: geometry collision mesh filename=package://my_jearm_moveit_config/config/meshes/right/r_link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; visual mesh filename=package://my_jearm_moveit_config/config/meshes/right/r_link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
- link Link7: geometry collision mesh filename=package://my_jearm_moveit_config/config/meshes/right/r_link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; visual mesh filename=package://my_jearm_moveit_config/config/meshes/right/r_link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
Joints:
- joint joint1: limit lower=-3.14 upper=3.14 effort=100 velocity=3.14 -> lower=-5.14 upper=5.14 effort=100 velocity=3.14
- joint joint2: limit lower=-1.85 upper=1.8 effort=100 velocity=3.14 -> lower=-1.86 upper=1.82 effort=100 velocity=3.14; origin xyz=0 0 0 rpy=-1.5708 0 0 -> xyz=0 0 0 rpy=1.5708 0 0
- joint joint3: origin xyz=0 -0.2719 0 rpy=1.5708 0 0 -> xyz=0 -0.2719 0 rpy=-1.5708 0 0
- joint joint4: limit lower=-2.26 upper=1.82 effort=100 velocity=3.14 -> lower=-2.27 upper=1.8 effort=100 velocity=3.14; origin xyz=-0.008 0 0 rpy=-1.5708 0 0 -> xyz=-0.008 0 0 rpy=1.5708 0 0
- joint joint5: origin xyz=0.008 -0.2189 0 rpy=1.5708 0 0 -> xyz=0.008 -0.2189 0 rpy=-1.5708 0 0
- joint joint6: origin xyz=0 0 0 rpy=-1.5708 0 0 -> xyz=0 0 0 rpy=1.5708 0 0
- joint joint7: origin xyz=0 -0.124 0 rpy=1.5708 0 0 -> xyz=0 -0.124 0 rpy=-1.5708 0 0
